Commit message: added camera to urdf and starting to work on navigation

File: shoebot_description/urdf/shoebot.urdf.xacro (robot description, xacro)
@@ -3,4 +3,6 @@
   <xacro:include filename="$(find shoebot_description)/urdf/create_base.urdf.xacro" />
   <xacro:include filename="$(find shoebot_description)/urdf/shoebot_gazebo.urdf.xacro" />
+  <xacro:include filename="$(find realsense2_description)/urdf/_d435.urdf.xacro" />
+  <xacro:arg name="use_nominal_extrinsics" default="True" />
   <xacro:create_base wheel_separation="0.235" base_diameter="0.3485">
     <mesh filename="package://shoebot_description/meshes/shoebot_collision.stl" scale="0.001 0.001 0.001" />
@@ -18,3 +20,6 @@
       <child link="laser_link" />
   </joint>
+  <xacro:sensor_d435 parent="base_link">
+    <origin xyz="0.045 0 0.078" rpy="0 0 0"/>
+  </xacro:sensor_d435>
 </robot>
