Commit message: working on urdf

File: shoebot_description/urdf/create_base.urdf.xacro (robot description, xacro)
@@ -53,5 +53,5 @@
     </inertial>
     <visual>
-      <origin xyz=" 0 0 0.0308" rpy="0 0 0" />
+      <origin xyz=" 0 0 -0.0308" rpy="1.57079 0 1.57079" />
       <geometry>
         <xacro:insert_block name="mesh" />

File: shoebot_description/urdf/shoebot.urdf.xacro (robot description, xacro)
@@ -4,5 +4,17 @@
   <xacro:include filename="$(find shoebot_description)/urdf/shoebot_gazebo.urdf.xacro" />
   <xacro:create_base wheel_separation="0.235" base_diameter="0.3485">
-    <mesh filename="package://shoebot_description/meshes/shoebot.dae" />
+    <mesh filename="package://shoebot_description/meshes/shoebot_collision.stl" scale="0.001 0.001 0.001" />
   </xacro:create_base>
+  <link name="laser_link" >
+      <inertial>
+      <mass value="0.01" />
+      <origin xyz="0 0 0" />
+      <inertia ixx="0.001" ixy="0.0" ixz="0.0" iyy="0.001" iyz="0.0" izz="0.001" />
+    </inertial>
+  </link>
+  <joint name="base_to_laser_joint" type="fixed">
+      <origin xyz="0 0 0.13" rpy="0 0 0" />
+      <parent link="base_link" />
+      <child link="laser_link" />
+  </joint>
 </robot>

Commit message: adding gazebo supportings

File: shoebot_description/urdf/create_base.urdf.xacro (robot description, xacro)
@@ -201,5 +201,5 @@
     <xacro:sim_create_wall_sensor/>
     <xacro:sim_create_cliff_sensors/>
-    <xacro:sim_imu/>
+    <!-- <xacro:sim_imu/> -->
   </xacro:macro>
 </robot>

File: shoebot_description/urdf/create_base_gazebo.urdf.xacro (robot description, xacro)
@@ -6,22 +6,22 @@
         <alwaysOn>true</alwaysOn>
         <updateRate>${diffdrive_update_rate}</updateRate>
-        <leftJoint>left_wheel_joint</leftJoint>
-        <rightJoint>right_wheel_joint</rightJoint>
-        <wheelSeparation>${wheel_separation}</wheelSeparation>
-        <wheelDiameter>${wheel_radius * 2}</wheelDiameter>
-        <wheelTorque>${wheel_torque}</wheelTorque>
+        <left_joint>left_wheel_joint</left_joint>
+        <right_joint>right_wheel_joint</right_joint>
+        <wheel_separation>${wheel_separation}</wheel_separation>
+        <wheel_diameter>${wheel_radius * 2}</wheel_diameter>
+        <wheel_torque>${wheel_torque}</wheel_torque>
         <!--wheelAcceleration>${wheel_accel}</wheelAcceleration-->
-        <commandTopic>cmd_vel</commandTopic>
-        <odometryTopic>odom</odometryTopic>
-        <odometryFrame>odom</odometryFrame>
-        <robotBaseFrame>base_footprint</robotBaseFrame>
+        <command_topic>cmd_vel</command_topic>
+        <odometry_topic>odom</odometry_topic>
+        <odometry_frame>odom</odometry_frame>
+        <robot_base_frame>base_footprint</robot_base_frame>
       </plugin>
       <plugin name="p3d_base_controller" filename="libgazebo_ros_p3d.so">
-        <alwaysOn>true</alwaysOn>
-        <updateRate>100.0</updateRate>
-        <bodyName>base_link</bodyName>
-        <topicName>simple_controller/absolute_position</topicName>
-        <gaussianNoise>0</gaussianNoise>
-        <frameName>map</frameName>
+        <always_on>true</always_on>
+        <update_rate>100.0</update_rate>
+        <body_name>base_link</body_name>
+        <topic_name>simple_controller/absolute_position</topic_name>
+        <gaussian_noise>0</gaussian_noise>
+        <frame_name>map</frame_name>
         <xyzOffsets>0 0 0</xyzOffsets>
         <rpyOffsets>0 0 0</rpyOffsets>
@@ -60,18 +60,4 @@
       <minDepth>0.001</minDepth>
       <maxVel>1.0</maxVel>
-    </gazebo>
-  </xacro:macro>
-  <xacro:macro name="sim_imu">
-    <gazebo>
-      <plugin name="imu_controller" filename="libgazebo_ros_imu.so">
-        <alwaysOn>true</alwaysOn>
-        <updateRate>30</updateRate>
-        <bodyName>gyro_link</bodyName>
-        <topicName>imu/data</topicName>
-        <serviceName>imu/is_calibrated</serviceName>
-        <gaussianNoise>${0.0017*0.0017}</gaussianNoise>
-        <xyzOffsets>0 0 0</xyzOffsets>
-        <rpyOffsets>0 0 0</rpyOffsets>
-      </plugin>
     </gazebo>
   </xacro:macro>

File: shoebot_description/urdf/shoebot.urdf.xacro (robot description, xacro)
@@ -4,8 +4,10 @@
   <xacro:include filename="$(find shoebot_description)/urdf/shoebot_gazebo.urdf.xacro" />
   <xacro:include filename="$(find realsense2_description)/urdf/_d435.urdf.xacro" />
+  <xacro:include filename="$(find shoebot_description)/urdf/generic_laser.urdf.xacro" />
   <xacro:arg name="use_nominal_extrinsics" default="True" />
   <xacro:create_base wheel_separation="0.235" base_diameter="0.3485">
-    <mesh filename="package://shoebot_description/meshes/shoebot_collision.stl" scale="0.001 0.001 0.001" />
+    <mesh filename="$(find shoebot_description)/meshes/shoebot_collision.stl" scale="0.001 0.001 0.001" />
   </xacro:create_base>
+<!--
   <link name="laser_link" >
       <inertial>
@@ -19,5 +21,11 @@
       <parent link="base_link" />
       <child link="laser_link" />
-  </joint>
+  </joint> -->
+  <xacro:property name="laser_pose">
+    <origin xyz="0 0 0.13" rpy="0 0 0"/>
+  </xacro:property>
+  <xacro:generic_laser>
+    <xacro:insert_block name="laser_pose" />
+  </xacro:generic_laser>
   <xacro:sensor_d435 parent="base_link">
     <origin xyz="0.045 0 0.078" rpy="0 0 0"/>
